File: Eaglescheme/Lab1_oppgave2.sch (EAGLE design)
At the start: 38 parts, among them IC1 MEGA8-P, IC2 LM2937, IC3 MEGA8-P, IC4 LM2937, IC5 MEGA8-P, IC7 LM2937, Q1 16MHz

Commit message: 1.8.4 _ ADC
Connections:
- net +5V: now also IC5.AREF
